File: Micro_mouse_circuit/Micro_mouse_final/Micro_mouse_final.kicad_sch (KiCad schematic)
At the start: 49 parts, among them J1 Conn_02x16_Odd_Even, J2 USB_C_Receptacle_PowerOnly_6P, J3 Conn_01x02, U1 HUSB237-AA001-DN06R, U10 AMS1117-3.3, U11 TPS22917DBV, U12 TPS22917DBV, U2 SK22D15L5, U3 LM2596SX-5_0/NOPB, U4 TP4056_C382139, U5 SN74LVC1G3157DCKR, U6 INA219AxDCN, U7 MT3608, U8 L298N_C19922, U9 L298N_C19922

Commit message: 02/28 submission
Parts:
- removed C1: 1uF, symbol Device:C
- removed C2: 220uF, symbol Device:C
- removed C4, C9: C, symbol Device:C
- removed C8: 680uF, symbol Device:C
- removed D1: SS34_C8678, xxcustom_footprint:SMA_L4.3-W2.6-LS5.2-RD, symbol SS34_C8678:SS34_C8678
- removed D2: Green_LED, symbol Device:LED
- removed D3: Red_LED, symbol Device:LED
- removed D4: M7_C95872, footprint:SMA_L4.3-W2.6-LS5.2-RD, symbol M7_C95872:M7_C95872
- removed D6: D_Schottky, symbol Device:D_Schottky
- removed J1: Conn_02x16_Odd_Even, Connector_PinHeader_2.54mm:PinHeader_2x16_P2.54mm_Vertical, symbol Connector_Generic:Conn_02x16_Odd_Even
- removed J3: Conn_01x02, Connector_JST:JST_PH_S2B-PH-K_1x02_P2.00mm_Horizontal, symbol Connector_Generic:Conn_01x02
- removed R1: 75k, symbol Device:R_US
- removed R10, R11, R12, R13, R14, R15, R16, R9: R, symbol Device:R
- removed R2: 0.4, xxcustom_footprint:R0402, symbol Device:R_US
- removed R3: 0.4, symbol Device:R_US
- removed R4, R5: 1k, xxcustom_footprint:R0402, symbol Device:R_US
- removed R6: 2k, xxcustom_footprint:R0402, symbol Device:R_US
- removed R7: 6k, xxcustom_footprint:R0402, symbol Device:R_US
- removed R8: 0.2, xxcustom_footprint:R2512, symbol Device:R_Shunt
- removed U1: HUSB237-AA001-DN06R, xxcustom_footprint:TDFN-6_L2.0-W2.0-P0.65-TL-EP, symbol HUSB237-AA001-DN06R:HUSB237-AA001-DN06R
- removed U10: AMS1117-3.3, Package_TO_SOT_SMD:SOT-223-3_TabPin2, symbol Regulator_Linear:AMS1117-3.3
- removed U11, U12: TPS22917DBV, Package_TO_SOT_SMD:SOT-23-6, symbol Power_Management:TPS22917DBV
- removed U2: SK22D15L5, xxcustom_footprint:SW-TH_XKB_SK22D15L7, symbol SK22D15L5:SK22D15L5
- removed U3: LM2596SX-5_0/NOPB, xxcustom_footprint:TO-263-5_L10.2-W8.9-P1.70-TL, symbol LM2596SX-5_0/NOPB:LM2596SX-5_0/NOPB
- removed U4: TP4056_C382139, xxcustom_footprint:ESOP-8_L4.9-W3.9-P1.27-LS6.0-BL-EP, symbol TP4056_C382139:TP4056_C382139
- removed U5: SN74LVC1G3157DCKR, xxcustom_footprint:SC-70-6_L2.2-W1.3-P0.65-LS2.1-BR, symbol SN74LVC1G3157DCKR:SN74LVC1G3157DCKR
- removed U6: INA219AxDCN, Package_TO_SOT_SMD:SOT-23-8, symbol Sensor_Energy:INA219AxDCN
- removed U7: MT3608, Package_TO_SOT_SMD:SOT-23-6, symbol Regulator_Switching:MT3608
- removed U9: L298N_C19922, footprint:MULTIWATT-15_L19.6-W5.0-P1.27-L, symbol L298N_C19922:L298N_C19922
- added C1: CL31B105KBHNNNE, xxcustom_footprint:C1206, symbol CL31B105KBHNNNE:CL31B105KBHNNNE
- added C4: RVT220UF10V67RV0037, xxcustom_footprint:CAP-SMD_BD6.3-L6.6-W6.6-FD, symbol RVT220UF10V67RV0037:RVT220UF10V67RV0037
- added D2, D6: SS34_C8678, xxcustom_footprint:SMA_L4.3-W2.6-LS5.2-RD, symbol SS34_C8678:SS34_C8678
- added J1: Conn_01x02, Connector_JST:JST_PH_S2B-PH-K_1x02_P2.00mm_Horizontal, symbol Connector_Generic:Conn_01x02
- added J3: Conn_02x16_Odd_Even, Connector_PinHeader_2.54mm:PinHeader_2x16_P2.54mm_Vertical, symbol Connector_Generic:Conn_02x16_Odd_Even
- added LED1, LED2: KT-0603R, xxcustom_footprint:R0603, symbol KT-0603R:KT-0603R
- added R1, R2: 0.2, xxcustom_footprint:R2512, symbol Device:R_Shunt
- added R10: 0805W8F4702T5E, xxcustom_footprint:R0805, symbol 0805W8F4702T5E:0805W8F4702T5E
- added R11: 0.4, xxcustom_footprint:R0402, symbol Device:R_US
- added R12: 2k, xxcustom_footprint:C1206, symbol Device:R_US
- added R14, R16: 1k, xxcustom_footprint:R0402, symbol Device:R_US
- added R15: 6k, xxcustom_footprint:R0805, symbol Device:R_US
- added R17, R18, R6: 10k, xxcustom_footprint:C1206, symbol Device:R
- added R3: 0603WAF7502T5E, xxcustom_footprint:R0603, symbol 0603WAF7502T5E:0603WAF7502T5E
- added R4: 0805W8F2702T5E, xxcustom_footprint:R0805, symbol 0805W8F2702T5E:0805W8F2702T5E
- added R5, R7, R8: 47k, xxcustom_footprint:R0805, symbol Device:R
- added REF1: high_frequency_680uF35V, xxcustom_footprint:CAP-TH_BD10.0-P5.00-D1.0-FD, symbol high_frequency_680uF35V:high_frequency_680uF35V
- added TP1, TP2, TP3, TP4, TP5: TestPoint, TestPoint:TestPoint_Pad_2.5x2.5mm, symbol Connector:TestPoint
- added U1: INA219AxDCN, Package_TO_SOT_SMD:SOT-23-8, symbol Sensor_Energy:INA219AxDCN
- added U10: SN74LVC1G3157DCKR, xxcustom_footprint:SC-70-6_L2.2-W1.3-P0.65-LS2.1-BR, symbol SN74LVC1G3157DCKR:SN74LVC1G3157DCKR
- added U11, U13: TPS22917DBVR, xxcustom_footprint:SOT-23-6_L2.9-W1.6-P0.95-LS2.8-BR, symbol TPS22917DBVR:TPS22917DBVR
- added U2: AMS1117-3.3, Package_TO_SOT_SMD:SOT-223-3_TabPin2, symbol Regulator_Linear:AMS1117-3.3
- added U3: HUSB237-AA001-DN06R, xxcustom_footprint:TDFN-6_L2.0-W2.0-P0.65-TL-EP, symbol HUSB237-AA001-DN06R:HUSB237-AA001-DN06R
- added U4: MT3608, xxcustom_footprint:SOT-23-6_L2.9-W1.6-P0.95-LS2.8-BL, symbol Regulator_Switching:MT3608
- added U5: LM2596SX-5_0/NOPB, xxcustom_footprint:TO-263-5_L10.2-W8.9-P1.70-TL, symbol LM2596SX-5_0/NOPB:LM2596SX-5_0/NOPB
- added U6: SK22D15L5, xxcustom_footprint:SW-TH_XKB_SK22D15L7, symbol SK22D15L5:SK22D15L5
- added U7: L298N_C19922, xxcustom_footprint:MULTIWATT-15_L19.6-W5.0-P1.27-L, symbol L298N_C19922:L298N_C19922
- added U9: TP4056_C382139, xxcustom_footprint:ESOP-8_L4.9-W3.9-P1.27-LS6.0-BL-EP, symbol TP4056_C382139:TP4056_C382139
- C3: value 10uF -> 22uF; footprint (none) -> xxcustom_footprint:C1206
- C5: value C -> 22uF; footprint (none) -> xxcustom_footprint:C1206
- C6: value C -> 22u; footprint (none) -> xxcustom_footprint:C1206
- C7: value C -> 10u; footprint (none) -> xxcustom_footprint:CAP-SMD_L3.2-W1.6-RD-C7171
- J2: footprint (none) -> xxcustom_footprint:TYPE-C-SMD_TYPE-C-6P
- L2, L3: value 10uH -> 10u
- L4: value L -> 10u; footprint (none) -> xxcustom_footprint:L0805
- U8: footprint footprint:MULTIWATT-15_L19.6-W5.0-P1.27-L -> xxcustom_footprint:MULTIWATT-15_L19.6-W5.0-P1.27-L
Connections:
- net 3V3 oUT: now also J3.18 (Pin_18)
- net 5V: now also L4.2, C4.1, R11.1, R2.4, U1.4 (VS), U1.8 (A1), U10.5 (VCC), U5.4 (FB), U9.8 (CE); no longer L3.2
- net 5V Out: now also J3.20 (Pin_20)
- net 5VBoosted: now also D6.1 (K), R5.1, TP1.1, U7.4 (VS), U7.9 (VSS)
- net 9V: now also C1.1, J3.22 (Pin_22), U3.2 (VUSB), U6.1
- net Battery: now also J3.14 (Pin_14)
- net BatteryPos: now also C7.1, R1.4, TP4.1, TP5.1, U6.5, U9.5 (BAT)
- net CTRL_EXT_LOAD1: now also J3.25 (Pin_25), U13.1 (VIN), U13.3 (ON)
- net CTRL_EXT_LOAD2: now also J3.7 (Pin_7), U11.1 (VIN), U11.3 (ON)
- net EXT_LOAD1_OUT: now also J3.21 (Pin_21), U13.6 (VOUT)
- net EXT_LOAD2_OUT: now also J3.11 (Pin_11), U11.6 (VOUT)
- net FAST_CHARGE_CTRL: now also J3.13 (Pin_13), U10.6 (S)
- net GND: now also C1.2, C4.2, D2.2 (A), J1.2 (Pin_2), J3.19 (Pin_19), J3.23 (Pin_23), R10.2, R12.1, R15.1, R17.1, R18.1, R3.2, R5.2, R6.1, R6.2, R7.1, R8.1, REF1.2, TP2.1, TP3.1, U1.3 (GND), U1.7 (A0), U10.2 (GND), U11.2 (GND), U13.2 (GND), U3.7 (GND), U4.2 (GND), U4.3 (FB), U5.3 (GND), U5.5 (ON#/OFF), U5.6 (GND), U7.8 (GND), U9.1 (TEMP), U9.3 (GND)
- net I2C1_SCL: now also J3.16 (Pin_16), U1.5 (SCL)
- net I2C1_SDA: now also J3.17 (Pin_17), U1.6 (SDA)
- net MOTOR1_A_OUT: now also J3.32 (Pin_32), U7.2 (OUT_1); no longer U8.2 (OUT_1)
- net MOTOR1_B_OUT: now also J3.31 (Pin_31), U7.3 (OUT_2); no longer U8.3 (OUT_2)
- net MOTOR1_CTRL1: now also J3.28 (Pin_28), U7.5 (Input_1); no longer U8.5 (Input_1)
- net MOTOR1_CTRL2: now also J3.30 (Pin_30), U7.7 (Input_2); no longer U8.7 (Input_2)
- net MOTOR2_CTRL1: now also U8.5 (Input_1), J3.4 (Pin_4)
- net MOTOR2_CTRL2: now also U8.7 (Input_2), J3.6 (Pin_6)
- net MOTOR3_A_OUT: now also J3.27 (Pin_27), U7.13 (Out3); no longer U8.13 (Out3)
- net MOTOR3_B_OUT: now also J3.29 (Pin_29), U7.14 (Out4); no longer U8.14 (Out4)
- net MOTOR3_CTRL1: now also J3.24 (Pin_24), U7.10 (Input_3); no longer U8.10 (Input_3)
- net MOTOR3_CTRL2: now also J3.26 (Pin_26), U7.12 (Input_4); no longer U8.12 (Input_4)
- net MOTOR4_CTRL1: now also U8.10 (Input_3), J3.8 (Pin_8)
- net MOTOR4_CTRL2: now also U8.12 (Input_4), J3.10 (Pin_10)
- net Motor2_A_OUT: now also U8.2 (OUT_1), J3.2 (Pin_2)
- net Motor2_B_OUT: now also U8.3 (OUT_2), J3.1 (Pin_1)
- net Motor4_A_OUT: now also U8.13 (Out3), J3.3 (Pin_3)
- net Motor4_B_Out: now also U8.14 (Out4), J3.5 (Pin_5)
- net R_prog: now also U10.4 (A), U9.2 (PROG)
- net SwitchCommon: now also L2.1, D2.1 (K), REF1.1, U5.1 (VIN), U5.2 (OUTPUT), U6.2
- net SwitchOn: now also C3.1, L1.1, U4.5 (IN), U6.6; no longer L4.1
- net USART2_RX: now also J3.9 (Pin_9)
- net USART2_TX: now also J3.12 (Pin_12)
- net V3.3Reg: now also R4.1, U2.2 (VO)
- net VBoost: now also U2.3 (VI)
- net at L3.1: now also L4.1; no longer L2.1
- net at L1.2: now also D6.2 (A), U4.1 (SW); no longer L2.2
- net at J2.A5 (CC1): now also U3.1 (CC1)
- net at J2.B5 (CC2): now also U3.6 (CC2)
- net at U8.1 (Sense_A): now also R18.2
- net at U8.15 (Sense_B): now also R7.2
- new net: R3.1, U3.3 (VSET)
- new net: R17.2, U7.1 (Sense_A)
- new net: R14.1, U9.6 (STDBY#)
- new net: LED2.1 (K), R14.2
- new net: R15.2, U10.3 (B1)
- new net: R11.2, U9.4 (VCC)
- new net: R16.2, U9.7 (CHRG#)
- new net: R1.2, U1.1 (IN+)
- new net: R1.3, U1.2 (IN-)
- new net: LED1.1 (K), R16.1
- new net: LED1.2 (A), LED2.2 (A), R2.1
- new net: R10.1, R4.2, U2.1 (GND)
- new net: L2.2, L3.2
- new net: R12.2, U10.1 (B2)
- new net: R8.2, U7.15 (Sense_B)
- new net: J1.1 (Pin_1), R1.1

Commit message: common share
Parts:
- removed R11: 0.4, xxcustom_footprint:R0402, symbol Device:R_US
- added R9: 0, xxcustom_footprint:C1206, symbol Device:R
- L1: value 10uH -> 10u
- R10: value 0805W8F4702T5E -> 47k
- R12, R17, R6: footprint xxcustom_footprint:C1206 -> xxcustom_footprint:R1206
- R14, R16: footprint xxcustom_footprint:R0402 -> xxcustom_footprint:R1206
- R15: value 6k -> 5.6k
- R3: value 0603WAF7502T5E -> 75k
- R4: value 0805W8F2702T5E -> 27k
Connections:
- net 5V: now also U9.4 (VCC), R9.1, R9.2
Changed lines of the file:
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@@
 	)
 	(junction
+		(at 226.06 50.8)
+		(diameter 0)
+		(color 0 0 0 0)
+	)
+	(junction
 		(at 125.73 101.6)
 		(diameter 0)
@@
 	)
 	(junction
+		(at 255.27 34.29)
+		(diameter 0)
+		(color 0 0 0 0)
+	)
+	(junction
 		(at 252.73 46.99)
 		(diameter 0)
@@
 	(wire
 		(pts
+			(xy 213.36 22.86) (xy 213.36 50.8)
+		)
+		(stroke
+			(width 0)
+			(type default)
+		)
+	)
+	(wire
+		(pts
 			(xy 54.61 38.1) (xy 58.42 38.1)
 		)
@@
 	(wire
 		(pts
-			(xy 252.73 34.29) (xy 255.27 34.29)
+			(xy 213.36 50.8) (xy 226.06 50.8)
 		)
 		(stroke
@@
 	(wire
 		(pts
+			(xy 226.06 50.8) (xy 226.06 57.15)
+		)
+		(stroke
+			(width 0)
+			(type default)
+		)
+	)
+	(wire
+		(pts
 			(xy 267.97 59.69) (xy 273.05 59.69)
 		)
@@
 	(wire
 		(pts
-			(xy 227.33 36.83) (xy 218.44 36.83)
+			(xy 227.33 36.83) (xy 219.71 36.83)
 		)
 		(stroke
@@
 	(wire
 		(pts
-			(xy 226.06 49.53) (xy 226.06 57.15)
+			(xy 226.06 41.91) (xy 226.06 50.8)
 		)
 		(stroke
@@
 	(wire
 		(pts
-			(xy 218.44 36.83) (xy 218.44 25.4)
+			(xy 219.71 36.83) (xy 219.71 30.48)
 		)
 		(stroke
@@
 	(wire
 		(pts
+			(xy 264.16 34.29) (xy 266.7 34.29)
+		)
+		(stroke
+			(width 0)
+			(type default)
+		)
+	)
+	(wire
+		(pts
+			(xy 255.27 34.29) (xy 255.27 22.86)
+		)
+		(stroke
+			(width 0)
+			(type default)
+		)
+	)
+	(wire
+		(pts
 			(xy 101.6 99.06) (xy 102.87 99.06)
 		)
@@
 		)
 	)
+	(wire
+		(pts
+			(xy 213.36 22.86) (xy 255.27 22.86)
+		)
+		(stroke
+			(width 0)
+			(type default)
+		)
+	)
+	(wire
+		(pts
+			(xy 252.73 34.29) (xy 255.27 34.29)
+		)
+		(stroke
+			(width 0)
+			(type default)
+		)
+	)
 	(polyline
 		(pts
@@
 	(wire
 		(pts
+			(xy 255.27 34.29) (xy 256.54 34.29)
+		)
+		(stroke
+			(width 0)
+			(type default)
+		)
+	)
+	(wire
+		(pts
 			(xy 43.18 191.77) (xy 27.94 191.77)
 		)
@@
 	)
 	(label "5V"
-		(at 255.27 34.29 0)
+		(at 266.7 34.29 0)
 		(effects
 			(font
@@
 	)
 	(label "R_prog"
-		(at 218.44 25.4 0)
+		(at 219.71 30.48 0)
 		(effects
 			(font
@@
 			)
 		)
-		(property "Description" "Resistor"
+		(property "Description" "Resistor C17902"
 			(at 201.93 232.41 0)
 			(effects
@@
 	)
 	(symbol
+		(lib_id "Device:R")
+		(at 260.35 34.29 90)
+		(unit 1)
+		(exclude_from_sim no)
+		(in_bom yes)
+		(on_board yes)
+		(dnp no)
+		(fields_autoplaced yes)
+		(property "Reference" "R9"
+			(at 260.35 27.94 90)
+			(effects
+				(font
+					(size 1.27 1.27)
+				)
+			)
+		)
+		(property "Value" "0"
+			(at 260.35 30.48 90)
+			(effects
+				(font
+					(size 1.27 1.27)
+				)
+			)
+		)
+		(property "Footprint" "xxcustom_footprint:C1206"
+			(at 260.35 36.068 90)
+			(effects
+				(font
+					(size 1.27 1.27)
+				)
+				(hide yes)
+			)
+		)
+		(property "Datasheet" "https://jlcpcb.com/parts/componentSearch?searchTxt=47k%CE%A9"
+			(at 260.35 34.29 0)
+			(effects
+				(font
+					(size 1.27 1.27)
+				)
+				(hide yes)
+			)
+		)
+		(property "Description" "Resistor"
+			(at 260.35 34.29 0)
+			(effects
+				(font
+					(size 1.27 1.27)
+				)
+				(hide yes)
+			)
+		)
+		(pin "2"
+		)
+		(pin "1"
+		)
+		(instances
+			(project "Micro_mouse_final"
+				(path "/0476620a-14c2-42c7-a46f-854d17e2e160"
+					(reference "R9")
+					(unit 1)
+				)
+			)
+		)
+	)
+	(symbol
 		(lib_id "TPS22917DBVR:TPS22917DBVR")
 		(at 307.34 181.61 0)
@@
 			)
 		)
-		(property "Value" "0603WAF7502T5E"
+		(property "Value" "75k"
 			(at 77.47 52.0699 90)
 			(effects
@@
 			)
 		)
-		(property "Footprint" "xxcustom_footprint:C1206"
+		(property "Footprint" "xxcustom_footprint:R1206"
 			(at 201.93 182.118 90)
 			(effects
@@
 			)
 		)
-		(property "Description" "Resistor"
+		(property "Description" "Resistor C17902"
 			(at 201.93 180.34 0)
 			(effects
@@
 			)
 		)
-		(property "Footprint" "xxcustom_footprint:R0402"
+		(property "Footprint" "xxcustom_footprint:R1206"
 			(at 263.906 43.434 90)
 			(effects
@@
 			)
 		)
-		(property "Value" "6k"
+		(property "Value" "5.6k"
 			(at 262.89 90.17 90)
 			(effects
@@
 			)
 		)
-		(property "Datasheet" "~"
+		(property "Datasheet" "C4382"
 			(at 262.89 93.98 0)
 			(effects
@@
 		(on_board yes)
 		(dnp no)
-		(fields_autoplaced yes)
 		(property "Reference" "C3"
-			(at 91.44 154.9399 0)
+			(at 81.534 155.194 0)
 			(effects
 				(font
@@
 		)
 		(property "Value" "22uF"
-			(at 91.44 157.4799 0)
+			(at 81.534 157.734 0)
 			(effects
 				(font
@@
 			)
 		)
-		(property "Description" "USB Power-Only 6P Type-C Receptacle connector"
+		(property "Description" "USB Power-Only 6P Type-C Receptacle connector: C5187463"
 			(at 39.37 45.72 0)
 			(effects
@@
 			)
 		)
-		(property "Value" "10uH"
+		(property "Value" "10u"
 			(at 100.33 146.05 90)
 			(effects
@@
 			)
 		)
-		(property "Value" "0805W8F4702T5E"
+		(property "Value" "47k"
 			(at 90.17 247.6499 90)
 			(effects
@@
 			)
 		)
-		(property "Description" ""
+		(property "Description" "0805W8F4702T5E"
 			(at 87.63 246.38 0)
 			(effects
@@
 	)
 	(symbol
-		(lib_id "Device:R_US")
-		(at 226.06 45.72 180)
-		(unit 1)
-		(exclude_from_sim no)
-		(in_bom yes)
-		(on_board yes)
-		(dnp no)
-		(property "Reference" "R11"
-			(at 221.742 44.704 0)
-			(effects
-				(font
-					(size 1.27 1.27)
-				)
-				(justify right)
-			)
-		)
-		(property "Value" "0.4"
-			(at 221.742 47.244 0)
-			(effects
-				(font
-					(size 1.27 1.27)
-				)
-				(justify right)
-			)
-		)
-		(property "Footprint" "xxcustom_footprint:R0402"
-			(at 225.044 45.466 90)
-			(effects
-				(font
-					(size 1.27 1.27)
-				)
-				(hide yes)
-			)
-		)
-		(property "Datasheet" "~"
-			(at 226.06 45.72 0)
-			(effects
-				(font
-					(size 1.27 1.27)
-				)
-				(hide yes)
-			)
-		)
-		(property "Description" "Resistor, US symbol"
-			(at 226.06 45.72 0)
-			(effects
-				(font
-					(size 1.27 1.27)
-				)
-				(hide yes)
-			)
-		)
-		(pin "2"
-		)
-		(pin "1"
-		)
-		(instances
-			(project "Micro_mouse_final"
-				(path "/0476620a-14c2-42c7-a46f-854d17e2e160"
-					(reference "R11")
-					(unit 1)
-				)
-			)
-		)
-	)
-	(symbol
 		(lib_id "power:GND")
 		(at 266.7 102.87 0)
@@
 			)
 		)
-		(property "Datasheet" "https://jlcpcb.com/parts/componentSearch?searchTxt=47k%CE%A9"
+		(property "Datasheet" "https://jlcpcb.com/partdetail/18401-0805W8F4702T5E/C17713"
 			(at 111.76 165.1 0)
 			(effects
@@
 			)
 		)
-		(property "Footprint" "xxcustom_footprint:C1206"
+		(property "Footprint" "xxcustom_footprint:R1206"
 			(at 244.094 92.964 90)
 			(effects
@@
 			)
 		)
-		(property "Datasheet" "~"
+		(property "Datasheet" "~C17944"
 			(at 243.84 93.98 0)
 			(effects
@@
 			)
 		)
-		(property "Value" "0805W8F2702T5E"
+		(property "Value" "27k"
 			(at 90.17 233.6799 90)
 			(effects
@@
 			)
 		)
-		(property "Description" ""
+		(property "Description" "0805W8F2702T5E"
 			(at 87.63 232.41 0)
 			(effects
@@
 			)
 		)
-		(property "Footprint" "xxcustom_footprint:C1206"
+		(property "Footprint" "xxcustom_footprint:R1206"
 			(at 109.982 175.26 90)
 			(effects
@@
 			)
 		)
-		(property "Footprint" "xxcustom_footprint:R0402"
+		(property "Footprint" "xxcustom_footprint:R1206"
 			(at 272.034 40.386 90)
 			(effects
@@
 			)
 		)
-		(property "Datasheet" "~"
+		(property "Datasheet" "~C459674"
 			(at 33.02 101.6 0)
 			(effects

Commit message: push  - kt
Parts:
- removed R2: 0.2, xxcustom_footprint:R2512, symbol Device:R_Shunt
- removed R9: 0, xxcustom_footprint:C1206, symbol Device:R
- removed REF1: high_frequency_680uF35V, xxcustom_footprint:CAP-TH_BD10.0-P5.00-D1.0-FD, symbol high_frequency_680uF35V:high_frequency_680uF35V
- added C2: 680u, xxcustom_footprint:CAP-TH_BD8.0-P3.50-D0.6-FD, symbol SPT1EM681F12OR:SPT1EM681F12OR
- added J4: Conn_01x01_Pin, symbol Connector:Conn_01x01_Pin
- added R11, R13, R9: 1, xxcustom_footprint:R1206, symbol 1206W4F100KT5E:1206W4F100KT5E
- added TP6, TP7, TP8, TP9: TestPoint, TestPoint:TestPoint_Pad_2.5x2.5mm, symbol Connector:TestPoint
- C1: value CL31B105KBHNNNE -> 1u
- C4: value RVT220UF10V67RV0037 -> 220u
Connections:
- net 5V: now also LED1.2 (A), LED2.2 (A), J4.1 (Pin_1), R11.1, R11.2, R13.1, R13.2, R9.1, R9.2, TP7.1
- net GND: now also C2.2, TP9.1; no longer R12.1, R15.1
- net R_prog: now also R12.1, R15.1; no longer U10.4 (A)
- net SwitchCommon: now also C2.1, TP6.1
- net at R3.1, U3.3 (VSET): now also TP8.1
- net VBoost renamed 5VBoost
Other:
- moved on the sheet: C4, L2, L3, L4, R3, U3

Commit message: FInal Additions to Schematic
-Added Kill Switch
-Moderated 3.3 Motor Control to 2.4 V
Parts:
- removed R17: 10k, xxcustom_footprint:R1206, symbol Device:R
- removed R18: 10k, xxcustom_footprint:C1206, symbol Device:R
- removed R7, R8: 47k, xxcustom_footprint:R0805, symbol Device:R
- removed TP2, TP3: TestPoint, TestPoint:TestPoint_Pad_2.5x2.5mm, symbol Connector:TestPoint
- added C8: 22u, xxcustom_footprint:C1206, symbol Device:C
- added R17, R20, R7, R8: RC-MT08W3R0JT, XXmicromouse:RES-ARRAY-SMD_0402-8P-L2.0-W1.0-BL, symbol 3OhmResistorArray:RC-MT08W3R0JT
- added R18, R2, R22, R24, R25, R27, R28, R30, R31, R33, R34, R36, R37, R39, R40, R42, R43: 27k, xxcustom_footprint:R0805, symbol 0805W8F2702T5E:0805W8F2702T5E
- added R19, R21, R23, R26, R29, R32, R35, R38, R41: 47k, xxcustom_footprint:R0805, symbol 0805W8F4702T5E:0805W8F4702T5E
- added U12: AMS1117-3.3, Package_TO_SOT_SMD:SOT-223-3_TabPin2, symbol Regulator_Linear:AMS1117-3.3
- added U14: SK22D15L5, xxcustom_footprint:SW-TH_XKB_SK22D15L7, symbol SK22D15L5:SK22D15L5
- R5: value 47k -> 8.2k; footprint xxcustom_footprint:R0805 -> XXmicromouse:R0805
- R6: value 10k -> 1.2K
- U2: footprint Package_TO_SOT_SMD:SOT-223-3_TabPin2 -> XXmicromouse:SOT-223-3_L6.5-W3.4-P2.30-LS7.0-BR
Connections:
- net 5VBoost is gone; now on net 5V Out: C6.1, U2.3 (VI)
- net 5VBoosted is gone; now on net 5V Out: C5.1, D6.1 (K), R5.1, TP1.1, U7.4 (VS), U7.9 (VSS), U8.4 (VS), U8.9 (VSS)
- net V3.3Reg is gone; now on net 3V3 OUT: R4.1, U2.2 (VO)
- net 5V: now also C8.1, U12.3 (VI); no longer U1.4 (VS), U1.8 (A1)
- net 5V Out: now also U1.4 (VS), U1.8 (A1)
- net BatteryPos: now also U14.4
- net GND: now also C8.2, R17.6, R19.2, R20.6, R22.2, R25.2, R28.2, R31.2, R34.2, R37.2, R40.2, R43.2, R7.1, R8.1; no longer R5.2, R6.1, U4.3 (FB), U5.5 (ON#/OFF)
- net MOTOR1_CTRL1: now also R38.1; no longer U7.5 (Input_1)
- net MOTOR1_CTRL2: now also R41.1; no longer U7.7 (Input_2)
- net MOTOR2_CTRL1: now also R21.1; no longer U8.5 (Input_1)
- net MOTOR2_CTRL2: now also R23.1; no longer U8.7 (Input_2)
- net MOTOR3_CTRL1: now also R32.1; no longer U7.10 (Input_3)
- net MOTOR3_CTRL2: now also R35.1; no longer U7.12 (Input_4)
- net MOTOR4_CTRL1: now also R26.1; no longer U8.10 (Input_3)
- net MOTOR4_CTRL2: now also R29.1; no longer U8.12 (Input_4)
- net at U8.1 (Sense_A): now also R7.4
- net at U8.15 (Sense_B): now also R20.5
- net at U7.1 (Sense_A): now also R8.4
- net 5VBoostedOn: now reaches U4.4 (EN)
- net 5VBoostedOn: now also U14.5
- net at U7.15 (Sense_B): now also R17.5
- net 3V3 oUT renamed 3V3 OUT
- net 3V3 OUT: now also R2.1, U12.2 (VO)
- new net: R20.3, R20.4
- new net: R27.2, R28.1
- new net: R18.2, R22.1
- new net: R42.2, R43.1
- new net: R39.2, R40.1
- new net: R33.2, R34.1
- new net: R19.1, R2.2, U12.1 (GND)
- new net: R17.3, R17.4
- new net: R5.2, R6.1, U4.3 (FB)
- new net: R36.2, R37.1
- new net: R24.2, R25.1
- new net: R7.2, R7.3
- new net: R7.5, R7.6
- new net: R7.7, R7.8
- new net: R30.2, R31.1
- new net: R8.2, R8.3
- new net: R8.5, R8.6
- new net: R8.7, R8.8
- new net 5V Regulator Off: U14.2, U5.5 (ON#/OFF)
- new net MOTOR1_CTRL1_2.4: R38.2, R39.1, U7.5 (Input_1)
- new net MOTOR1_CTRL2_2.4: R41.2, R42.1, U7.7 (Input_2)
- new net MOTOR2_CTRL1_2.4: R18.1, R21.2, U8.5 (Input_1)
- new net MOTOR2_CTRL2_2.4: R23.2, R24.1, U8.7 (Input_2)
- new net MOTOR3_CTRL1_2.4: R32.2, R33.1, U7.10 (Input_3)
- new net MOTOR3_CTRL2_2.4: R35.2, R36.1, U7.12 (Input_4)
- new net MOTOR4_CTRL1_2.4: R26.2, R27.1, U8.10 (Input_3)
- new net MOTOR4_CTRL2_2.4: R29.2, R30.1, U8.12 (Input_4)
Other:
- note added: "-5A"
- note added: "-5B"
- note added: "3.3->2.4 Voltage divider"
- note added: "3.3V Off"
- note added: "4D"
- note added: "9V"
- note added: "M1- Back, Left Driver"
- note added: "M3 - Back Left Auxillary"
- note added: "Master Kill Switch"
- note added: "Off"
- note added: "On"
- note removed: "Motor 1 - Motor 4"
- note removed: "Need to find suitable configuration of capacitors"
- moved on the sheet: C6, R10, R4, U11, U13, U2, U7, U8
